File: mark4-fc/indicators.kicad_sch (KiCad schematic)
At the start: 10 parts, among them Q1 SS8050

Commit message: feat(hardware): shrink mark4-fc to 36x36 and split assembly by side
Board outline, connectors and assembly strategy all move in one pass;
schematic, PCB and the fab package are propagated together.

- Rebuild the Edge.Cuts outline at 36x36 (the floor the 30.5 mm M3
  pattern allows) and fix the four corner fillets whose arc midpoints
  sat diametrically opposite, which cut a 4 mm disc out of each corner.
- Reduce SWD from 6 to 3 positions (SWDIO/SWCLK/GND) so SWD plus USB-C
  fit the edge budget; SWO is gone, BOOT0 stays the recovery path.
- Move the hand-soldered parts (LDO, flash, Q1, JP1, test points and
  their pull-ups) to the bottom face; the JLCPCB package now covers the
  top side only (CPL 63 -> 52, BOM 31 -> 26 lines).
- Re-relax the placement into the smaller outline with the electrically
  critical groups hand-anchored (crystal, VCAP, buck corner, connector
  ESD); LED strip pads move to the left edge to clear the USB row.
  DRC clean, schematic parity 0, nothing routed yet.
- Hide top-silk refdes and values in favour of pad labels, add the
  orientation arrow (direction still to confirm against the frame).
- Replace the footprint-family CPL rotation table with measured,
  LCSC-keyed corrections (jlcpcb-cpl-rotations.csv), derived from the
  EasyEDA footprints; fixes U2, U1 and Q1 which the community table got
  wrong or missed.
- Correct the STO-2 flash substitution note: no 256 Mbit Winbond exists
  in SOIC-8 208 mil; list the real drop-ins and the EN4B firmware cost.

Co-Authored-By: Claude Fable 5 <noreply@anthropic.com>
Parts:
- R13, R14, R15: MPN (none) -> 0603WAF1001T5E
- R16: MPN (none) -> 0603WAF1002T5E
Changed lines of the file:
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@@
+			)
+		)
+		(property "MPN" "0603WAF1001T5E"
+			(at 53.34 149.86 0)
+			(hide yes)
+			(show_name no)
+			(do_not_autoplace no)
+			(effects
+				(font
+					(size 1.27 1.27)
+				)
 			)
 		)
@@
 			)
 		)
-    (property "MPN" "NCD0603Y2" (at 101.6 101.6 0)
-      (effects (font (size 1.27 1.27)) (hide yes))
-    )
+		(property "MPN" "NCD0603Y2"
+			(at 101.6 101.6 0)
+			(hide yes)
+			(show_name no)
+			(do_not_autoplace no)
+			(effects
+				(font
+					(size 1.27 1.27)
+				)
+			)
+		)
 		(pin "1"
 		)
@@
 			)
 		)
+		(property "MPN" "0603WAF1001T5E"
+			(at 88.9 101.6 0)
+			(hide yes)
+			(show_name no)
+			(do_not_autoplace no)
+			(effects
+				(font
+					(size 1.27 1.27)
+				)
+			)
+		)
 		(property "Notes" "LED2 series resistor. 1k at 3V3 gives about 1.0-1.7 mA into D5 (NCD0603Y2 yellow), roughly 10-25 mcd."
 			(at 88.9 101.6 0)
@@
 			)
 		)
+		(property "MPN" "0603WAF1001T5E"
+			(at 88.9 88.9 0)
+			(hide yes)
+			(show_name no)
+			(do_not_autoplace no)
+			(effects
+				(font
+					(size 1.27 1.27)
+				)
+			)
+		)
 		(property "Notes" "LED1 series resistor. 1k at 3V3 gives about 1.0-1.7 mA into D4 (KT-0603R red), roughly 10-25 mcd."
 			(at 88.9 88.9 0)
@@
 			)
 		)
+		(property "MPN" "0603WAF1002T5E"
+			(at 60.96 156.21 0)
+			(hide yes)
+			(show_name no)
+			(do_not_autoplace no)
+			(effects
+				(font
+					(size 1.27 1.27)
+				)
+			)
+		)
 		(property "Notes" "Base-to-GND pull-down: keeps the buzzer silent while PB5 is high-Z at reset."
 			(at 60.96 156.21 0)
@@
 			)
 		)
-    (property "MPN" "0805W8F510KT5E" (at 76.2 127.0 0)
-      (effects (font (size 1.27 1.27)) (hide yes))
-    )
+		(property "MPN" "0805W8F510KT5E"
+			(at 76.2 127 0)
+			(hide yes)
+			(show_name no)
+			(do_not_autoplace no)
+			(effects
+				(font
+					(size 1.27 1.27)
+				)
+			)
+		)
 		(pin "1"
 		)
@@
 			)
 		)
-    (property "MPN" "KT-0603R" (at 101.6 88.9 0)
-      (effects (font (size 1.27 1.27)) (hide yes))
-    )
+		(property "MPN" "KT-0603R"
+			(at 101.6 88.9 0)
+			(hide yes)
+			(show_name no)
+			(do_not_autoplace no)
+			(effects
+				(font
+					(size 1.27 1.27)
+				)
+			)
+		)
 		(pin "1"
 		)
