File: mark4-fc/mcu.kicad_sch (KiCad schematic)
At the start: 21 parts, among them J1 SWD, U3 STM32F722RETx, Y1 8MHz

Commit message: feat(hardware): shrink mark4-fc to 36x36 and split assembly by side
Board outline, connectors and assembly strategy all move in one pass;
schematic, PCB and the fab package are propagated together.

- Rebuild the Edge.Cuts outline at 36x36 (the floor the 30.5 mm M3
  pattern allows) and fix the four corner fillets whose arc midpoints
  sat diametrically opposite, which cut a 4 mm disc out of each corner.
- Reduce SWD from 6 to 3 positions (SWDIO/SWCLK/GND) so SWD plus USB-C
  fit the edge budget; SWO is gone, BOOT0 stays the recovery path.
- Move the hand-soldered parts (LDO, flash, Q1, JP1, test points and
  their pull-ups) to the bottom face; the JLCPCB package now covers the
  top side only (CPL 63 -> 52, BOM 31 -> 26 lines).
- Re-relax the placement into the smaller outline with the electrically
  critical groups hand-anchored (crystal, VCAP, buck corner, connector
  ESD); LED strip pads move to the left edge to clear the USB row.
  DRC clean, schematic parity 0, nothing routed yet.
- Hide top-silk refdes and values in favour of pad labels, add the
  orientation arrow (direction still to confirm against the frame).
- Replace the footprint-family CPL rotation table with measured,
  LCSC-keyed corrections (jlcpcb-cpl-rotations.csv), derived from the
  EasyEDA footprints; fixes U2, U1 and Q1 which the community table got
  wrong or missed.
- Correct the STO-2 flash substitution note: no 256 Mbit Winbond exists
  in SOIC-8 208 mil; list the real drop-ins and the EN4B firmware cost.

Co-Authored-By: Claude Fable 5 <noreply@anthropic.com>
Parts:
- J1: footprint Connector_PinHeader_2.54mm:PinHeader_1x06_P2.54mm_Vertical -> Connector_PinHeader_2.54mm:PinHeader_1x03_P2.54mm_Vertical; symbol Connector_Generic:Conn_01x06 -> Connector_Generic:Conn_01x03; Notes Not assembled - hand-populated 3 pins (GND, SWCLK, SWDIO), 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 -> Not assembled - hand-populated 3 pins, SWDIO / SWCLK / GND
- R3: MPN (none) -> 0603WAF1002T5E
Connections:
- net +3V3: no longer J1.1 (Pin_1)
- net NRST: no longer J1.5 (Pin_5)
- net SWDIO: now also J1.1 (Pin_1); no longer J1.4 (Pin_4)
- net LED_DATA: now reaches U3.43 (PA10)
- net PWR_SRC: now reaches U3.53 (PC12)
- net 12V_SENSE renamed VBAT_SENSE
- net SWO: no longer names the net of U3.55 (PB3)
- net SWO: no longer J1.6 (Pin_6)
- no-connect marks 11 -> 10
Other:
- note added: "Not on this sheet: the I2C1 4.7k pull-ups on PB8/PB9 (sensor sheet), the 10k pull-up on FLASH_CS/PB12 (storage sheet, the W25Q /CS must track VCC at power-up), the VBAT divider and its Schottky feeding VBAT_SENSE (power sheet, PWR-4), and the USB 90 ohm pair plus ESD array on USB_DM/USB_DP (USB sheet, CON-5, no series resistors). PA4 and PA5 are TTa pins (3.3 V max): nothing 5 V may ever touch IM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"
- note removed: "Not on this sheet: the I2C1 4.7k pull-ups on PB8/PB9 (sensor sheet), the 10k pull-up on FLASH_CS/PB12 (storage sheet, the W25Q /CS must track VCC at power-up), the 12 V divider and its Schottky feeding 12V_SENSE (power sheet, PWR-4), and the USB 90 ohm pair plus ESD array on USB_DM/USB_DP (USB sheet, CON-5, no series resistors). PA4 and PA5 are TTa pins (3.3 V max): nothing 5 V may ever touch IMU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"
Changed lines of the file:
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@@
 		)
 	)
-	(text "Not on this sheet: the I2C1 4.7k pull-ups on PB8/PB9 (sensor sheet), the 10k pull-up on\nFLASH_CS/PB12 (storage sheet, the W25Q /CS must track VCC at power-up), the 12 V divider\nand its Schottky feeding 12V_SENSE (power sheet, PWR-4), and the USB 90 ohm pair plus ESD\narray on USB_DM/USB_DP (USB sheet, CON-5, no series resistors).\nPA4 and PA5 are TTa pins (3.3 V max): nothing 5 V may ever touch IMU_CS or SPI1_SCK."
+	(text "Not on this sheet: the I2C1 4.7k pull-ups on PB8/PB9 (sensor sheet), the 10k pull-up on\nFLASH_CS/PB12 (storage sheet, the W25Q /CS must track VCC at power-up), the VBAT divider\nand its Schottky feeding VBAT_SENSE (power sheet, PWR-4), and the USB 90 ohm pair plus ESD\narray on USB_DM/USB_DP (USB sheet, CON-5, no series resistors).\nPA4 and PA5 are TTa pins (3.3 V max): nothing 5 V may ever touch IMU_CS or SPI1_SCK."
 		(exclude_from_sim no)
 		(at 250 216 0)
@@
 	)
 	(no_connect
-		(at 179.07 160.02)
-	)
-	(no_connect
 		(at 179.07 139.7)
 	)
 	(no_connect
-		(at 219.71 134.62)
-	)
-	(no_connect
 		(at 219.71 132.08)
 	)
@@
 	(wire
 		(pts
-			(xy 294.64 134.62) (xy 283.21 134.62)
-		)
-		(stroke
-			(width 0)
-			(type default)
-		)
-	)
-	(wire
-		(pts
 			(xy 219.71 129.54) (xy 250.19 129.54)
 		)
@@
 	(wire
 		(pts
-			(xy 280.67 139.7) (xy 280.67 154.94)
+			(xy 280.67 142.24) (xy 280.67 154.94)
 		)
 		(stroke
@@
 	(wire
 		(pts
-			(xy 294.64 139.7) (xy 280.67 139.7)
+			(xy 294.64 142.24) (xy 280.67 142.24)
 		)
 		(stroke
@@
 	(wire
 		(pts
-			(xy 283.21 134.62) (xy 283.21 127)
-		)
-		(stroke
-			(width 0)
-			(type default)
-		)
-	)
-	(wire
-		(pts
 			(xy 93.98 175.26) (xy 101.6 175.26)
 		)
@@
 	)
 	(label "NRST"
-		(at 294.64 144.78 180)
-		(effects
-			(font
-				(size 1.27 1.27)
-			)
-			(justify right bottom)
-		)
-	)
-	(label "NRST"
 		(at 179.07 109.22 180)
 		(effects
@@
 		)
 	)
-	(label "SWO"
-		(at 294.64 147.32 180)
-		(effects
-			(font
-				(size 1.27 1.27)
-			)
-			(justify right bottom)
-		)
-	)
 	(label "OSC_OUT"
 		(at 179.07 121.92 180)
@@
 		)
 	)
-	(label "SWO"
-		(at 219.71 160.02 0)
-		(effects
-			(font
-				(size 1.27 1.27)
-			)
-			(justify left bottom)
-		)
-	)
-	(label "SWDIO"
-		(at 294.64 142.24 180)
-		(effects
-			(font
-				(size 1.27 1.27)
-			)
-			(justify right bottom)
-		)
+(no_connect
+		(at 219.71 160.02)
 	)
 	(label "BOOT0"
@@
 	)
 	(label "SWCLK"
+		(at 294.64 139.7 180)
+		(effects
+			(font
+				(size 1.27 1.27)
+			)
+			(justify right bottom)
+		)
+	)
+	(label "SWDIO"
 		(at 294.64 137.16 180)
 		(effects
@@
 		)
 	)
-	(hierarchical_label "12V_SENSE"
+	(hierarchical_label "VBAT_SENSE"
 		(shape input)
 		(at 179.07 132.08 180)
@@
 		)
 	)
+	(hierarchical_label "LED_DATA"
+		(shape output)
+		(at 219.71 134.62 0)
+		(effects
+			(font
+				(size 1.27 1.27)
+			)
+			(justify left)
+		)
+	)
+	(hierarchical_label "PWR_SRC"
+		(shape input)
+		(at 179.07 160.02 180)
+		(effects
+			(font
+				(size 1.27 1.27)
+			)
+			(justify right)
+		)
+	)
 	(hierarchical_label "M3"
 		(shape output)
@@
 			)
 		)
-    (property "MPN" "CL21A475KAQNNNE" (at 200.66 72.39 0)
-      (effects (font (size 1.27 1.27)) (hide yes))
-    )
+		(property "MPN" "CL21A475KAQNNNE"
+			(at 200.66 72.39 0)
+			(hide yes)
+			(show_name no)
+			(do_not_autoplace no)
+			(effects
+				(font
+					(size 1.27 1.27)
+				)
+			)
+		)
 		(pin "1"
 		)
@@
 			)
 		)
+		(property "MPN" "0603WAF1002T5E"
+			(at 72.39 154.94 0)
+			(hide yes)
+			(show_name no)
+			(do_not_autoplace no)
+			(effects
+				(font
+					(size 1.27 1.27)
+				)
+			)
+		)
 		(pin "1"
 		)
@@
 			)
 		)
-    (property "MPN" "0603CG8R2C500NT" (at 77.47 185.42 0)
-      (effects (font (size 1.27 1.27)) (hide yes))
-    )
+		(property "MPN" "0603CG8R2C500NT"
+			(at 77.47 185.42 0)
+			(hide yes)
+			(show_name no)
+			(do_not_autoplace no)
+			(effects
+				(font
+					(size 1.27 1.27)
+				)
+			)
+		)
 		(pin "1"
 		)
@@
 			)
 		)
-    (property "MPN" "CL10A105KB8NNNC" (at 238.76 72.39 0)
-      (effects (font (size 1.27 1.27)) (hide yes))
-    )
-		(pin "1"
-		)
-		(pin "2"
-		)
-		(instances
-			(project "mark4-fc"
-				(path "/30be79cb-0cbd-4664-b75b-d8a85c58cd22/91613667-32a2-42b2-aeba-8646756e1841"
-					(reference "C15")
-					(unit 1)
-				)
-			)
-		)
-	)
-	(symbol
-		(lib_id "power:+3V3")
-		(at 283.21 127 0)
-		(unit 1)
-		(body_style 1)
-		(exclude_from_sim no)
-		(in_bom yes)
-		(on_board yes)
-		(in_pos_files yes)
-		(dnp no)
-		(property "Reference" "#PWR112"
-			(at 283.21 123.19 0)
-			(hide yes)
-			(show_name no)
-			(do_not_autoplace no)
-			(effects
-				(font
-					(size 1.27 1.27)
-				)
-			)
-		)
-		(property "Value" "+3V3"
-			(at 283.21 130.556 0)
-			(show_name no)
-			(do_not_autoplace no)
-			(effects
-				(font
-					(size 1.27 1.27)
-				)
-			)
-		)
-		(property "Footprint" ""
-			(at 283.21 127 0)
-			(hide yes)
-			(show_name no)
-			(do_not_autoplace no)
-			(effects
-				(font
-					(size 1.27 1.27)
-				)
-			)
-		)
-		(property "Datasheet" ""
-			(at 283.21 127 0)
-			(hide yes)
-			(show_name no)
-			(do_not_autoplace no)
-			(effects
-				(font
-					(size 1.27 1.27)
-				)
-			)
-		)
-		(property "Description" "Power symbol creates a global label with name +3V3"
-			(at 283.21 127 0)
+		(property "MPN" "CL10A105KB8NNNC"
+			(at 238.76 72.39 0)
 			(hide yes)
 			(show_name no)
@@
 		(pin "1"
 		)
+		(pin "2"
+		)
 		(instances
 			(project "mark4-fc"
 				(path "/30be79cb-0cbd-4664-b75b-d8a85c58cd22/91613667-32a2-42b2-aeba-8646756e1841"
-					(reference "#PWR112")
+					(reference "C15")
 					(unit 1)
 				)
@@
 			)
 		)
-    (property "MPN" "0603CG8R2C500NT" (at 101.6 185.42 0)
-      (effects (font (size 1.27 1.27)) (hide yes))
-    )
+		(property "MPN" "0603CG8R2C500NT"
+			(at 101.6 185.42 0)
+			(hide yes)
+			(show_name no)
+			(do_not_autoplace no)
+			(effects
+				(font
+					(size 1.27 1.27)
+				)
+			)
+		)
 		(pin "1"
 		)
@@
 			)
 		)
-    (property "MPN" "CL21A475KAQNNNE" (at 167.64 177.8 0)
-      (effects (font (size 1.27 1.27)) (hide yes))
-    )
+		(property "MPN" "CL21A475KAQNNNE"
+			(at 167.64 177.8 0)
+			(hide yes)
+			(show_name no)
+			(do_not_autoplace no)
+			(effects
+				(font
+					(size 1.27 1.27)
+				)
+			)
+		)
 		(pin "1"
 		)
@@
 	)
 	(symbol
-		(lib_id "Connector_Generic:Conn_01x06")
+		(lib_id "Connector_Generic:Conn_01x03")
 		(at 299.72 139.7 0)
 		(unit 1)
@@
 		(dnp no)
 		(property "Reference" "J1"
-			(at 299.72 147.32 0)
+			(at 299.72 134.62 0)
 			(show_name no)
 			(do_not_autoplace no)
@@
 		)
 		(property "Value" "SWD"
-			(at 299.72 129.54 0)
+			(at 299.72 144.78 0)
 			(show_name no)
 			(do_not_autoplace no)
@@
 			)
 		)
-		(property "Footprint" "Connector_PinHeader_2.54mm:PinHeader_1x06_P2.54mm_Vertical"
+		(property "Footprint" "Connector_PinHeader_2.54mm:PinHeader_1x03_P2.54mm_Vertical"
 			(at 299.72 139.7 0)
 			(hide yes)
@@
 			)
 		)
-		(property "Description" "Generic connector, single row, 01x06, script generated (kicad-library-utils/schlib/autogen/connector/)"
+		(property "Description" "Generic connector, single row, 01x03, script generated (kicad-library-utils/schlib/autogen/connector/)"
 			(at 299.72 139.7 0)
 			(hide yes)
@@
 			)
 		)
-		(property "Notes" "Not assembled - hand-populated 3 pins (GND, SWCLK, SWDIO), all 6 positions routed"
+		(property "Notes" "Not assembled - hand-populated 3 pins, SWDIO / SWCLK / GND"
 			(at 299.72 139.7 0)
 			(hide yes)
@@
 		(pin "3"
 		)
-		(pin "4"
-		)
-		(pin "5"
-		)
-		(pin "6"
-		)
 		(instances
