File: mark4-fc/power.kicad_sch (KiCad schematic)
At the start: 15 parts, among them U1 AP63205WU, U2 TLV1117LV33

Commit message: feat(hardware): shrink mark4-fc to 36x36 and split assembly by side
Board outline, connectors and assembly strategy all move in one pass;
schematic, PCB and the fab package are propagated together.

- Rebuild the Edge.Cuts outline at 36x36 (the floor the 30.5 mm M3
  pattern allows) and fix the four corner fillets whose arc midpoints
  sat diametrically opposite, which cut a 4 mm disc out of each corner.
- Reduce SWD from 6 to 3 positions (SWDIO/SWCLK/GND) so SWD plus USB-C
  fit the edge budget; SWO is gone, BOOT0 stays the recovery path.
- Move the hand-soldered parts (LDO, flash, Q1, JP1, test points and
  their pull-ups) to the bottom face; the JLCPCB package now covers the
  top side only (CPL 63 -> 52, BOM 31 -> 26 lines).
- Re-relax the placement into the smaller outline with the electrically
  critical groups hand-anchored (crystal, VCAP, buck corner, connector
  ESD); LED strip pads move to the left edge to clear the USB row.
  DRC clean, schematic parity 0, nothing routed yet.
- Hide top-silk refdes and values in favour of pad labels, add the
  orientation arrow (direction still to confirm against the frame).
- Replace the footprint-family CPL rotation table with measured,
  LCSC-keyed corrections (jlcpcb-cpl-rotations.csv), derived from the
  EasyEDA footprints; fixes U2, U1 and Q1 which the community table got
  wrong or missed.
- Correct the STO-2 flash substitution note: no 256 Mbit Winbond exists
  in SOIC-8 208 mil; list the real drop-ins and the EN4B firmware cost.

Co-Authored-By: Claude Fable 5 <noreply@anthropic.com>
Parts:
- removed D1, D2: SS54, Diode_SMD:D_SMA, symbol Device:D_Schottky
- added C26: 22uF, Capacitor_SMD:C_0805_2012Metric, symbol Device:C
- added R18: 100k, Resistor_SMD:R_0603_1608Metric, symbol Device:R
- added R19: 33k, Resistor_SMD:R_0603_1608Metric, symbol Device:R
- added R20: 10k, Resistor_SMD:R_0603_1608Metric, symbol Device:R
- added U8: TPS2116DRL, Package_TO_SOT_SMD:SOT-583-8, symbol Power_Management:TPS2116DRL
- R1: value 10k -> 100k; LCSC C25804 -> C25803; MPN 0603WAF1002T5E -> 0603WAF1003T5E
- R2: value 1.5k -> 12k; LCSC C22843 -> C22790; MPN 0603WAF1501T5E -> 0603WAF1202T5E
Connections:
- net +3V3: now also R20.1
- net +5V: now also C26.1, U8.2 (VOUT), U8.7 (VOUT)
- net GND: now also C26.2, R19.2, U8.1 (GND)
- net VBUS: now also U8.6 (VIN2)
- net +12V renamed +10V
- net +10V: no longer R1.1
- net 12V_SENSE renamed VBAT_SENSE
- net 5V_BUCK renamed +5V_BUCK
- net +5V_BUCK: now also R18.1, U8.3 (VIN1), U8.5 (MODE)
- new net: R18.2, R19.1, U8.4 (PR1)
- new net PWR_SRC: R20.2, U8.8 (ST)
- new net VBAT: R1.1
Other:
- note added: "10 V BEC input and 5 V buck (PWR-1)"
- note added: "5 V active OR-ing / power mux (PWR-3)"
- note added: "The board is fed from the ESC BEC and never from raw VBAT: motor braking spikes on a 6S pack can exceed the 32 V input rating of the AP63205, and the BEC absorbs them. Measured source: T-Motor Velox 45A V2, 10 V BEC."
- note added: "The divider now hangs on the raw battery instead of a regulated rail, so pack voltage is directly visible; the old input-rail divider could not see it. R1/R2 = 100k/12k, ratio 12/112 = 0.10714. Tap = 2.70 V at 25.2 V (6S max), 1.80 V at 16.8 V (4S max), and 3.3 V (VDDA) is reached only at 30.8 V, so any plausible pack transient stays inside the ADC range. Drain 0.22 mA continuous while the pack i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"
- note added: "U1 is the fixed 5 V version: FB is tied to the buck output (5V_BUCK) per the datasheet, and EN is tied to VIN (always on). OR stage: D1 also blocks the AP63205 high-side body diode, so USB power on the shared rail cannot back-feed the 10 V net (PWR-3)."
- note added: "U8 replaces the two Schottky ORing diodes: 40 mOhm typical (60 mOhm over temperature) instead of 300 mV of drop, and it blocks in BOTH legs, so USB 5 V cannot back-drive the AP63205 output through its high-side body diode. MODE tied to VIN1 selects priority mode: the BEC wins whenever it is there, so plugging or unplugging USB never disturbs a board that is already flying. R18/R19 set the switcho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"
- note added: "VBAT sense to ADC, raw battery at the ESC pad group (PWR-4)"
- note removed: "12 V input and 5 V buck (PWR-1)"
- note removed: "12 V rail sense to ADC (PWR-4)"
- note removed: "5 V OR-ing (PWR-3)"
- note removed: "R1/R2 = 10k/1.5k, ratio 1.5/11.5 = 0.1304. Tap = 1.57 V at 12 V nominal, and reaches 3.3 V (VDDA) only at a 25.3 V rail, so the ADC input stays below VDDA for any plausible transient on the ESC 12 V rail. D3 clamps negative excursions: DS11853 Table 60 allows zero negative current injection on PC0..PC3."
- note removed: "U1 is the fixed 5 V version: FB is tied to the buck output (5V_BUCK) per the datasheet, and EN is tied to VIN (always on). OR stage: D1 also blocks the AP63205 high-side body diode, so USB power on the shared rail cannot back-feed the 12 V net (PWR-3)."
