File: mark4-fc/storage.kicad_sch (KiCad schematic)
At the start: 5 parts, among them U6 W25Q128JVSIQ

Commit message: feat(hardware): shrink mark4-fc to 36x36 and split assembly by side
Board outline, connectors and assembly strategy all move in one pass;
schematic, PCB and the fab package are propagated together.

- Rebuild the Edge.Cuts outline at 36x36 (the floor the 30.5 mm M3
  pattern allows) and fix the four corner fillets whose arc midpoints
  sat diametrically opposite, which cut a 4 mm disc out of each corner.
- Reduce SWD from 6 to 3 positions (SWDIO/SWCLK/GND) so SWD plus USB-C
  fit the edge budget; SWO is gone, BOOT0 stays the recovery path.
- Move the hand-soldered parts (LDO, flash, Q1, JP1, test points and
  their pull-ups) to the bottom face; the JLCPCB package now covers the
  top side only (CPL 63 -> 52, BOM 31 -> 26 lines).
- Re-relax the placement into the smaller outline with the electrically
  critical groups hand-anchored (crystal, VCAP, buck corner, connector
  ESD); LED strip pads move to the left edge to clear the USB row.
  DRC clean, schematic parity 0, nothing routed yet.
- Hide top-silk refdes and values in favour of pad labels, add the
  orientation arrow (direction still to confirm against the frame).
- Replace the footprint-family CPL rotation table with measured,
  LCSC-keyed corrections (jlcpcb-cpl-rotations.csv), derived from the
  EasyEDA footprints; fixes U2, U1 and Q1 which the community table got
  wrong or missed.
- Correct the STO-2 flash substitution note: no 256 Mbit Winbond exists
  in SOIC-8 208 mil; list the real drop-ins and the EN4B firmware cost.

Co-Authored-By: Claude Fable 5 <noreply@anthropic.com>
Parts:
- R10, R8, R9: MPN (none) -> 0603WAF1002T5E
Changed lines of the file:
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@@
+			)
+		)
+		(property "MPN" "0603WAF1002T5E"
+			(at 72.39 78.74 0)
+			(hide yes)
+			(show_name no)
+			(do_not_autoplace no)
+			(effects
+				(font
+					(size 1.27 1.27)
+				)
 			)
 		)
@@
 			)
 		)
+		(property "MPN" "0603WAF1002T5E"
+			(at 99.06 78.74 0)
+			(hide yes)
+			(show_name no)
+			(do_not_autoplace no)
+			(effects
+				(font
+					(size 1.27 1.27)
+				)
+			)
+		)
 		(property "Notes" "/CS pull-up (STO-1): the die has no internal one and the datasheet requires /CS to track VCC at power-up, when the MCU pin is still high-Z"
 			(at 99.06 78.74 0)
@@
 			(at 80.01 78.74 0)
 			(hide yes)
+			(show_name no)
+			(do_not_autoplace no)
+			(effects
+				(font
+					(size 1.27 1.27)
+				)
+			)
+		)
+		(property "MPN" "0603WAF1002T5E"
+			(at 80.01 78.74 0)
+			(hide yes)
